File: KiCAD/stickMk2-schematic/stickMk2-schematic.sch (KiCad schematic (older format))
At the start: 10 parts, among them J1 Conn_01x08, J2 Conn_01x08

Commit message: Added XTAL reference
Parts:
- added C? (x2): 3.3pF, symbol Device:C
- added Y?: 12MHz, symbol Device:Crystal_GND24
Connections:
- net GND: now also C?.1, C?.2, Y?.2, Y?.4
- net at U?.7 (XTAL1/PB6): now also C?.2, Y?.3
- net at U?.8 (XTAL2/PB7): now also C?.1, Y?.1
Other:
- moved on the sheet: J1, J2
Changed lines of the file:
@@
 P 6150 4300
 F 0 "R?" V 5943 4300 50  0001 C CNN
-F 1 "68R" V 6035 4300 50  0000 C CNN
+F 1 "68R" V 6250 4300 50  0000 C CNN
 F 2 "" V 6080 4300 50  0001 C CNN
 F 3 "~" H 6150 4300 50  0001 C CNN
@@
 U 1 1 60F834CD
 P 7800 4350
-F 0 "USB" H 7857 4725 50  0000 C CNN
+F 0 "USB" H 7700 4750 50  0000 C CNN
 F 1 "USB_A" H 7857 4726 50  0001 C CNN
 F 2 "" H 7950 4300 50  0001 C CNN
@@
 L Connector_Generic:Conn_01x08 J2
 U 1 1 60F99D93
-P 8000 2650
-F 0 "J2" H 8080 2596 50  0000 L CNN
-F 1 "Conn_01x08" H 8080 2551 50  0001 L CNN
-F 2 "" H 8000 2650 50  0001 C CNN
-F 3 "~" H 8000 2650 50  0001 C CNN
-	1    8000 2650
-	1    0    0    -1
-$EndComp
-Text GLabel 7800 2350 0    50   Input ~ 0
+P 8450 2650
+F 0 "J2" H 8400 3100 50  0000 L CNN
+F 1 "Conn_01x08" H 8530 2551 50  0001 L CNN
+F 2 "" H 8450 2650 50  0001 C CNN
+F 3 "~" H 8450 2650 50  0001 C CNN
+	1    8450 2650
+	1    0    0    -1
+$EndComp
+Text GLabel 8250 2350 0    50   Input ~ 0
 PD6LED
-Text GLabel 7800 2650 0    50   Input ~ 0
+Text GLabel 8250 2650 0    50   Input ~ 0
 SCK
-Text GLabel 7800 2750 0    50   Input ~ 0
+Text GLabel 8250 2750 0    50   Input ~ 0
 RST
-Text GLabel 7800 2850 0    50   Input ~ 0
+Text GLabel 8250 2850 0    50   Input ~ 0
 MISO
-Text GLabel 7800 2950 0    50   Input ~ 0
+Text GLabel 8250 2950 0    50   Input ~ 0
 MOSI
-Text GLabel 7800 3050 0    50   Input ~ 0
+Text GLabel 8250 3050 0    50   Input ~ 0
 PC1
 $Comp
 L power:GND #PWR?
 U 1 1 60F9C6CA
-P 7350 2550
-F 0 "#PWR?" H 7350 2300 50  0001 C CNN
-F 1 "GND" H 7355 2377 50  0001 C CNN
-F 2 "" H 7350 2550 50  0001 C CNN
-F 3 "" H 7350 2550 50  0001 C CNN
-	1    7350 2550
-	1    0    0    -1
-$EndComp
-Wire Wire Line
-	7800 2550 7350 2550
+P 7800 2550
+F 0 "#PWR?" H 7800 2300 50  0001 C CNN
+F 1 "GND" H 7805 2377 50  0001 C CNN
+F 2 "" H 7800 2550 50  0001 C CNN
+F 3 "" H 7800 2550 50  0001 C CNN
+	1    7800 2550
+	1    0    0    -1
+$EndComp
+Wire Wire Line
+	8250 2550 7800 2550
 $Comp
 L power:VCC #PWR?
 U 1 1 60F9CE61
-P 7350 2450
-F 0 "#PWR?" H 7350 2300 50  0001 C CNN
-F 1 "VCC" H 7365 2623 50  0000 C CNN
-F 2 "" H 7350 2450 50  0001 C CNN
-F 3 "" H 7350 2450 50  0001 C CNN
-	1    7350 2450
-	1    0    0    -1
-$EndComp
-Wire Wire Line
-	7800 2450 7350 2450
+P 7800 2450
+F 0 "#PWR?" H 7800 2300 50  0001 C CNN
+F 1 "VCC" H 7815 2623 50  0000 C CNN
+F 2 "" H 7800 2450 50  0001 C CNN
+F 3 "" H 7800 2450 50  0001 C CNN
+	1    7800 2450
+	1    0    0    -1
+$EndComp
+Wire Wire Line
+	8250 2450 7800 2450
 $Comp
 L Connector_Generic:Conn_01x08 J1
 U 1 1 60F9DB1B
-P 6950 2650
-F 0 "J1" H 7030 2596 50  0000 L CNN
-F 1 "Conn_01x08" H 7030 2551 50  0001 L CNN
-F 2 "" H 6950 2650 50  0001 C CNN
-F 3 "~" H 6950 2650 50  0001 C CNN
-	1    6950 2650
-	1    0    0    -1
-$EndComp
-Text GLabel 6750 2350 0    50   Input ~ 0
+P 7400 2650
+F 0 "J1" H 7350 3100 50  0000 L CNN
+F 1 "Conn_01x08" H 7480 2551 50  0001 L CNN
+F 2 "" H 7400 2650 50  0001 C CNN
+F 3 "~" H 7400 2650 50  0001 C CNN
+	1    7400 2650
+	1    0    0    -1
+$EndComp
+Text GLabel 7200 2350 0    50   Input ~ 0
 PB2
-Text GLabel 6750 2450 0    50   Input ~ 0
+Text GLabel 7200 2450 0    50   Input ~ 0
 PB1
-Text GLabel 6750 2550 0    50   Input ~ 0
+Text GLabel 7200 2550 0    50   Input ~ 0
 PB0
-Text GLabel 6750 2650 0    50   Input ~ 0
+Text GLabel 7200 2650 0    50   Input ~ 0
 PD7
-Text GLabel 6750 2750 0    50   Input ~ 0
+Text GLabel 7200 2750 0    50   Input ~ 0
 PD5
-Text GLabel 6750 2850 0    50   Input ~ 0
+Text GLabel 7200 2850 0    50   Input ~ 0
 PC4
-Text GLabel 6750 2950 0    50   Input ~ 0
+Text GLabel 7200 2950 0    50   Input ~ 0
 PC3
-Text GLabel 6750 3050 0    50   Input ~ 0
+Text GLabel 7200 3050 0    50   Input ~ 0
 PC2
+$Comp
+L Device:Crystal_GND24 Y?
+U 1 1 60F9F121
+P 6100 3200
+F 0 "Y?" V 6146 2956 50  0001 R CNN
+F 1 "12MHz" V 6300 3500 50  0000 R CNN
+F 2 "" H 6100 3200 50  0001 C CNN
+F 3 "~" H 6100 3200 50  0001 C CNN
+	1    6100 3200
+	0    -1   -1   0
+$EndComp
+$Comp
+L Device:C C?
+U 1 1 60FA7CA0
+P 6250 2800
+F 0 "C?" V 5998 2800 50  0001 C CNN
+F 1 "3.3pF" V 6090 2800 50  0000 C CNN
+F 2 "" H 6288 2650 50  0001 C CNN
+F 3 "~" H 6250 2800 50  0001 C CNN
+	1    6250 2800
+	0    1    1    0
+$EndComp
+$Comp
+L Device:C C?
+U 1 1 60FAC2F2
+P 6250 3650
+F 0 "C?" V 5998 3650 50  0001 C CNN
+F 1 "3.3pF" V 6410 3650 50  0000 C CNN
+F 2 "" H 6288 3500 50  0001 C CNN
+F 3 "~" H 6250 3650 50  0001 C CNN
+	1    6250 3650
+	0    -1   -1   0
+$EndComp
+Wire Wire Line
+	6100 3050 6100 2800
+Wire Wire Line
+	5900 3200 5800 3200
+$Comp
+L power:GND #PWR?
+U 1 1 60FAFF04
+P 5800 3300
+F 0 "#PWR?" H 5800 3050 50  0001 C CNN
+F 1 "GND" H 5805 3127 50  0001 C CNN
+F 2 "" H 5800 3300 50  0001 C CNN
+F 3 "" H 5800 3300 50  0001 C CNN
+	1    5800 3300
+	1    0    0    -1
+$EndComp
+Wire Wire Line
+	5800 3200 5800 3300
+Wire Wire Line
+	6100 3350 6100 3650
+Wire Wire Line
+	6100 3650 5600 3650
+Wire Wire Line
+	5600 3650 5600 3000
+Wire Wire Line
+	5600 3000 5250 3000
+Wire Wire Line
+	6100 2800 5600 2800
+Wire Wire Line
+	5600 2800 5600 2900
+Wire Wire Line
+	5600 2900 5250 2900
+Connection ~ 6100 2800
+$Comp
+L power:GND #PWR?
+U 1 1 60FB2B02
+P 6450 3700
+F 0 "#PWR?" H 6450 3450 50  0001 C CNN
+F 1 "GND" H 6455 3527 50  0001 C CNN
+F 2 "" H 6450 3700 50  0001 C CNN
+F 3 "" H 6450 3700 50  0001 C CNN
+	1    6450 3700
+	1    0    0    -1
+$EndComp
+Wire Wire Line
+	6400 3650 6450 3650
+Wire Wire Line
+	6450 3650 6450 3700
+Wire Wire Line
+	6300 3200 6450 3200
+Wire Wire Line
+	6450 3200 6450 3650
+Connection ~ 6450 3650
+Wire Wire Line
+	6400 2800 6450 2800
+Wire Wire Line
+	6450 2800 6450 3200
+Connection ~ 6450 3200
+Connection ~ 6100 3650
 $EndSCHEMATC
